File: hardware/SynthPass.kicad_pcb (KiCad board)
At the start: 4 copper layers, 19.1 x 16.8 mm, 18 parts, among them J1 SM04B-SRSS-TB, J2 USB_C_Receptacle_USB2.0_16P, SW1 SW_Push, U1 CH572D, Y1 32MHz

Commit message: Update back silk rev. # to track board revision
Other:
- board text added: "R${REVISION}"
- board text removed: "R1.1"
Changed lines of the file:
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@@
 		)
 	)
-	(gr_text "R1.1"
+	(gr_text "R${REVISION}"
 		(at 160.3 54 315)
 		(layer "B.SilkS")
